Commit message: Remove meshes from test directory

File: tests/data/franka_test.urdf (robot description, URDF)
Before this commit: robot franka, 12 links, 10 joints
Links:
- link franka_0_link0: geometry collision box size=0.227 0.2 0.141; visual box size=0.227 0.2 0.141
- link franka_0_link1: geometry collision box size=0.115 0.09 0.112; collision cylinder length=0.112 radius=0.0575
- link franka_0_link2: geometry collision box size=0.115 0.09 0.112; collision cylinder length=0.214 radius=0.0575
- link franka_0_link3: geometry collision box size=0.085 0.095 0.05; collision cylinder length=0.226 radius=0.0575
- link franka_0_link4: geometry collision box size=0.085 0.05 0.095; collision cylinder length=0.224 radius=0.0575
- link franka_0_link5: geometry collision box size=0.092 0.056 0.22; collision cylinder length=0.19 radius=0.0575
- link franka_0_link6: geometry collision box size=0.05 0.115 0.088; collision cylinder length=0.19 radius=0.049
- link franka_0_link7: geometry 
- link franka_0_link8: geometry collision box size=0.06 0.075 0.04; visual box size=0.06 0.075 0.04
- link franka_stand: geometry collision box size=1 1.5112 2.5; collision box size=1 1.5112 2.5
