Commit message: trying to fix up urdf with masses

File: tests/data/franka_test_with_mass.urdf (robot description, URDF)
Before this commit: robot franka, 52 links, 52 joints
Links:
- removed link camera_link
- removed link camera_rgb_optical_frame
- removed link cup
- removed link dispense
- removed link hotel_pan_sixth_6in_kisses
- removed link hotel_pan_sixth_6in_mnms
- removed link hotel_pan_sixth_6in_reeses
- removed link hotel_pan_sixth_6in_skittles
- removed link mobile_demo_cal_left
- removed link mobile_demo_cal_right
- removed link mobile_demo_frame
- removed link realsense_base_link
- removed link realsense_color_frame
- removed link realsense_color_optical_frame
- removed link realsense_depth_frame
- removed link realsense_depth_optical_frame
- removed link realsense_left_ir_frame
- removed link realsense_left_ir_optical_frame
- removed link realsense_link
- removed link realsense_right_ir_frame
- removed link realsense_right_ir_optical_frame
- removed link realsense_tag_alignment_frame
- removed link spoon_1oz_kisses_face
- removed link spoon_1oz_kisses_tag
- removed link spoon_1oz_kisses_tc
- removed link spoon_1oz_kisses_tip
- removed link spoon_1oz_mnms_face
- removed link spoon_1oz_mnms_tag
- removed link spoon_1oz_mnms_tc
- removed link spoon_1oz_mnms_tip
- removed link spoon_1oz_reeses_face
- removed link spoon_1oz_reeses_tag
- removed link spoon_1oz_reeses_tc
- removed link spoon_1oz_reeses_tip
- removed link spoon_1oz_skittles_face
- removed link spoon_1oz_skittles_tag
- removed link spoon_1oz_skittles_tc
- removed link spoon_1oz_skittles_tip
Joints:
- removed joint base_link_to_cup_joint
- removed joint base_link_to_mobile_demo_frame
- removed joint base_link_to_spoon_1oz_kisses_tc_joint
- removed joint base_link_to_spoon_1oz_mnms_tc_joint
- removed joint base_link_to_spoon_1oz_skittles_tc_joint
- removed joint camera_link_to_optical
- removed joint cup_to_cup_dispense
- removed joint feh_mate_to_spoon_1oz_reeses_tc_joint
- removed joint franka_feh_to_realsense_base_link
- removed joint global_to_mobile_demo_frame
- removed joint mobile_demo_frame_to_cal_left
- removed joint mobile_demo_frame_to_cal_right
- removed joint mobile_demo_frame_to_hotel_pan_sixth_6in_kisses
- removed joint mobile_demo_frame_to_hotel_pan_sixth_6in_mnms
- removed joint mobile_demo_frame_to_hotel_pan_sixth_6in_reeses
- removed joint mobile_demo_frame_to_hotel_pan_sixth_6in_skittles
- removed joint realsense_color_joint
- removed joint realsense_color_optical_joint
- removed joint realsense_color_tag_joint
- removed joint realsense_depth_joint
- removed joint realsense_depth_optical_joint
- removed joint realsense_depth_to_camera
- removed joint realsense_joint
- removed joint realsense_left_ir_joint
- removed joint realsense_left_ir_optical_joint
- removed joint realsense_right_ir_joint
- removed joint realsense_right_ir_optical_joint
- removed joint spoon_1oz_kisses_face_to_spoon_1oz_kisses_tip
- removed joint spoon_1oz_kisses_tc_to_spoon_1oz_kisses_face
- removed joint spoon_1oz_kisses_tc_to_spoon_1oz_kisses_tag
- removed joint spoon_1oz_mnms_face_to_spoon_1oz_mnms_tip
- removed joint spoon_1oz_mnms_tc_to_spoon_1oz_mnms_face
- removed joint spoon_1oz_mnms_tc_to_spoon_1oz_mnms_tag
- removed joint spoon_1oz_reeses_face_to_spoon_1oz_reeses_tip
- removed joint spoon_1oz_reeses_tc_to_spoon_1oz_reeses_face
- removed joint spoon_1oz_reeses_tc_to_spoon_1oz_reeses_tag
- removed joint spoon_1oz_skittles_face_to_spoon_1oz_skittles_tip
- removed joint spoon_1oz_skittles_tc_to_spoon_1oz_skittles_face
- removed joint spoon_1oz_skittles_tc_to_spoon_1oz_skittles_tag
- joint base_foot_world: origin xyz=0.0 0.0 0.0 rpy=0.0 0.0 0.0 -> xyz=0 0 0 rpy=0 0 0
