Commit message: - adding unit tests - updating joint limits of urdf

File: franka_robot_multibody_collision.urdf (robot description, URDF)
Before this commit: robot franka, 14 links, 13 joints
Joints:
- joint franka_joint1: limit lower=-2.8773 upper=2.8773 effort=87 velocity=2.1750 -> lower=-2.8973 upper=2.8973 effort=87 velocity=2.1750
- joint franka_joint2: limit lower=-1.7428 upper=1.7428 effort=87 velocity=2.1750 -> lower=-1.7628 upper=1.7628 effort=87 velocity=2.1750
- joint franka_joint3: limit lower=-2.8773 upper=2.8773 effort=87 velocity=2.1750 -> lower=-2.8973 upper=2.8973 effort=87 velocity=2.1750
- joint franka_joint4: limit lower=-3.0518 upper=-0.0898 effort=87 velocity=2.1750 -> lower=-3.0718 upper=-0.0698 effort=87 velocity=2.1750
- joint franka_joint5: limit lower=-2.8773 upper=2.8773 effort=12 velocity=2.6100 -> lower=-2.8973 upper=2.8973 effort=12 velocity=2.6100
- joint franka_joint6: limit lower=0.0075 upper=3.6825 effort=12 velocity=2.6100 -> lower=-0.0175 upper=3.7525 effort=12 velocity=2.6100
- joint franka_joint7: limit lower=-2.8773 upper=2.8773 effort=12 velocity=2.6100 -> lower=-2.8973 upper=2.8973 effort=12 velocity=2.6100

File: tests/data/franka_test.urdf (robot description, URDF)
Before this commit: robot franka, 12 links, 10 joints
Links:
- removed link base_footprint
- removed link franka_0_link0
- removed link franka_0_link1
- removed link franka_0_link2
- removed link franka_0_link3
- removed link franka_0_link4
- removed link franka_0_link5
- removed link franka_0_link6
- removed link franka_0_link7
- removed link franka_0_link8
- removed link franka_stand
- added link base_aa
- added link franka_head_js; collision cylinder length=0.08 radius=0.07; collision cylinder length=0.1 radius=0.05
- added link franka_link0; visual box size=0.227 0.2 0.141
- added link franka_link1; collision box size=0.115 0.09 0.112; collision cylinder length=0.112 radius=0.0825
- added link franka_link2; collision box size=0.115 0.09 0.112; collision cylinder length=0.214 radius=0.0575
- added link franka_link3; collision box size=0.085 0.095 0.05; collision cylinder length=0.226 radius=0.0575
- added link franka_link4; collision box size=0.085 0.05 0.095; collision cylinder length=0.224 radius=0.0575
- added link franka_link5; collision box size=0.092 0.056 0.22; collision cylinder length=0.19 radius=0.0575
- added link franka_link6; collision box size=0.05 0.115 0.088; collision cylinder length=0.19 radius=0.049
- added link franka_link7
- added link franka_link8; collision box size=0.06 0.075 0.04; visual box size=0.06 0.075 0.04
- added link tool; collision cylinder length=0.275 radius=0.041; visual cylinder length=0.275 radius=0.041
- added link tool_tip
Joints:
- removed joint base_foot_joint
- removed joint franka_0_joint1
- removed joint franka_0_joint2
- removed joint franka_0_joint3
- removed joint franka_0_joint4
- removed joint franka_0_joint5
- removed joint franka_0_joint6
- removed joint franka_0_joint7
- removed joint franka_0_joint8
- removed joint franka_0_joint_base_link
- added joint base_aa_joint: type fixed, parent base_link, child base_aa, origin xyz=0.01905 -0.04134 0.0 rpy=0 0 0
- added joint franka_head_to_tool_joint: type fixed, parent franka_head_js, child tool, origin xyz=0.0 0 0.075 rpy=0 0 0
- added joint franka_joint1: type revolute, parent franka_link0, child franka_link1, origin xyz=0 0 0.333 rpy=0 0 0, axis 0 0 1, limit lower=-2.8973 upper=2.8973 effort=87 velocity=2.1750
- added joint franka_joint2: type revolute, parent franka_link1, child franka_link2, origin xyz=0 0 0 rpy=-1.57079632679 0 0, axis 0 0 1, limit lower=-1.7628 upper=1.7628 effort=87 velocity=2.1750
- added joint franka_joint3: type revolute, parent franka_link2, child franka_link3, origin xyz=0 -0.316 0 rpy=1.57079632679 0 0, axis 0 0 1, limit lower=-2.8973 upper=2.8973 effort=87 velocity=2.1750
- added joint franka_joint4: type revolute, parent franka_link3, child franka_link4, origin xyz=0.0825 0 0 rpy=1.57079632679 0 0, axis 0 0 1, limit lower=-3.0718 upper=-0.0698 effort=87 velocity=2.1750
- added joint franka_joint5: type revolute, parent franka_link4, child franka_link5, origin xyz=-0.0825 0.384 0 rpy=-1.57079632679 0 0, axis 0 0 1, limit lower=-2.8973 upper=2.8973 effort=12 velocity=2.6100
- added joint franka_joint6: type revolute, parent franka_link5, child franka_link6, origin xyz=0 0 0 rpy=1.57079632679 0 0, axis 0 0 1, limit lower=-0.0175 upper=3.7525 effort=12 velocity=2.6100
- added joint franka_joint7: type revolute, parent franka_link6, child franka_link7, origin xyz=0.088 0 0 rpy=1.57079632679 0 0, axis 0 0 1, limit lower=-2.8973 upper=2.8973 effort=12 velocity=2.6100
- added joint franka_joint8: type fixed, parent franka_link7, child franka_link8, origin xyz=0 0 0.107 rpy=0 0 0, axis 0 0 0
- added joint franka_joint_base_aa: type fixed, parent base_aa, child franka_link0, origin xyz=0 0 0 rpy=0 0 1.5708
- added joint franka_link8_to_franka_head_js: type fixed, parent franka_link8, child franka_head_js, origin xyz=0.0 0.000 0.0075 rpy=0 0 0.785398
- added joint tool_joint_to_tool_tip: type fixed, parent tool, child tool_tip, origin xyz=0.0 0 0.275 rpy=0 0 0
